File: serial-switch-panel/serial-switch-panel.kicad_pcb (KiCad board)
At the start: 2 copper layers, 41.9 x 31.8 mm, 58 parts, among them J10 Conn_01x01, J11 Conn_01x01, J12 Conn_01x01, J13 Conn_01x01, J14 Conn_01x01, J15 Conn_01x01, J16 Conn_01x01, J17 Conn_01x01, J18 Conn_01x01, J2 2501551-4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

Commit message: [fp] Check/Finalize PCB
Routing:
- net +5V: track 38.0 -> 47.0 mm, vias 4 -> 6
Other:
- board text added: "LD"
- board text added: "PWR"
- board text added: "Power Control Input Board (C) Electronics Tinkerer 2026-03-07 v1.0A"
Changed lines of the file:
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@@
 		(embedded_fonts no)
+	)
+	(gr_circle
+		(center 103.81 87.06)
+		(end 107.112 87.06)
+		(stroke
+			(width 0.1524)
+			(type solid)
+		)
+		(fill no)
+		(layer "F.Cu")
+	)
+	(gr_circle
+		(center 103.81 111.19)
+		(end 107.112 111.19)
+		(stroke
+			(width 0.1524)
+			(type solid)
+		)
+		(fill no)
+		(layer "F.Cu")
+	)
+	(gr_circle
+		(center 138.1 111.19)
+		(end 141.402 111.19)
+		(stroke
+			(width 0.1524)
+			(type solid)
+		)
+		(fill no)
+		(layer "F.Cu")
 	)
 	(gr_rect
@@
 		(layer "Edge.Cuts")
 	)
+	(gr_text "PWR"
+		(at 110.3124 113.7424 0)
+		(layer "F.SilkS")
+		(effects
+			(font
+				(size 0.8 0.8)
+				(thickness 0.15)
+			)
+			(justify top)
+		)
+	)
+	(gr_text "LD"
+		(at 121.6408 113.7424 0)
+		(layer "F.SilkS")
+		(effects
+			(font
+				(size 0.8 0.8)
+				(thickness 0.15)
+			)
+			(justify top)
+		)
+	)
 	(gr_text "(+)"
 		(at 102.286 93.41 0)
@@
 				(thickness 0.15)
 			)
+		)
+	)
+	(gr_text "Power Control Input Board\n(C) Electronics Tinkerer\n2026-03-07 v1.0A"
+		(at 129.208 91.886 0)
+		(layer "B.SilkS")
+		(effects
+			(font
+				(size 1 1)
+				(thickness 0.15)
+			)
+			(justify mirror)
 		)
 	)
@@
 	)
 	(segment
+		(start 124.13 114.238)
+		(end 125.4 114.238)
+		(width 0.508)
+		(layer "F.Cu")
+		(net "+5V")
+	)
+	(segment
 		(start 129.21 113.285)
 		(end 131.065 113.285)
@@
 	)
 	(segment
+		(start 125.4 113.285)
+		(end 125.4 114.238)
+		(width 0.508)
+		(layer "F.Cu")
+		(net "+5V")
+	)
+	(segment
 		(start 132.525 111.825)
 		(end 132.525 109.998)
@@
 	)
 	(segment
+		(start 125.4 114.238)
+		(end 130.226 114.238)
+		(width 0.508)
+		(layer "F.Cu")
+		(net "+5V")
+	)
+	(segment
 		(start 128.1515 96.74)
 		(end 128.1515 96.2631)
@@
 	)
 	(via
+		(at 134.544 108.396)
+		(size 0.7)
+		(drill 0.3)
+		(layers "F.Cu" "B.Cu")
+		(free yes)
+		(net "+5V")
+	)
+	(via
 		(at 126.5176 103.5446)
 		(size 0.7)
@@
 		(net "+5V")
 	)
+	(via
+		(at 134.544 106.364)
+		(size 0.7)
+		(drill 0.3)
+		(layers "F.Cu" "B.Cu")
+		(free yes)
+		(net "+5V")
+	)
+	(segment
+		(start 134.544 106.364)
+		(end 134.544 108.396)
+		(width 0.508)
+		(layer "B.Cu")
+		(net "+5V")
+	)
