File: serial-relay-switch/serial-relay-switch.kicad_pcb (KiCad board)
At the start: 2 copper layers, 170.2 x 66 mm, 78 parts, among them J1 Screw_Terminal_01x01, J10 Screw_Terminal_01x01, J11 Screw_Terminal_01x01, J17 Conn_01x01, J18 Conn_01x01, J19 Screw_Terminal_01x01, J2 2501551-4, J20 Screw_Terminal_01x01, J21 Conn_01x01, J4 Screw_Terminal_01x01, J5 Screw_Terminal_01x01, J6 Screw_Terminal_01x01, J7 Screw_Terminal_01x01, J8 Screw_Terminal_01x01, J9 Screw_Terminal_01x01, K1 G2RL-1-E, K2 G2RL-1-E, K3 G2RL-1-E, K4 G2RL-1-E, K5 G2RL-1-E, K6 G2RL-1-E, K7 G2RL-1-E, K8 G2RL-1-E, U1 H11L1, U10 SZNUD3124LT1G, U11 SZNUD3124LT1G, U12 SZNUD3124LT1G, U13 74HCT595, U14 74LVC1G32, U15 74LVC1G08, U16 74LVC1G04, U17 74LS163, U2 ISL8488E, U3 SZNUD3124LT1G, U4 ISL8488E, U6 SZNUD3124LT1G, U7 SZNUD3124LT1G, U8 SZNUD3124LT1G, U9 SZNUD3124LT1G

Commit message: [rs] Ready for review
Routing:
- net /CLK: track 155.9 -> 133.5 mm
Other:
- outline, holes or cut-outs redrawn
Changed lines of the file:
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@@
 		(tags "capacitor")
 		(property "Reference" "C4"
-			(at 0 -1.43 0)
+			(at 2.667 0 0)
 			(layer "F.SilkS")
 			(effects
@@
 		(tags "Resistor Axial_DIN0414 series Axial Vertical pin pitch 5.08mm 2W length 11.9mm diameter 4.5mm")
 		(property "Reference" "R30"
-			(at 2.54 -3.37 90)
+			(at -3.319 0 180)
 			(layer "F.SilkS")
 			(effects
@@
 		(tags "D_SOD-123F")
 		(property "Reference" "D1"
-			(at 3.81 0 90)
+			(at 3.048 0 180)
 			(layer "F.SilkS")
 			(effects
@@
 	)
 	(gr_line
-		(start 78.41 101.03)
+		(start 78.41 97.982)
 		(end 78.41 106.11)
 		(stroke
@@
 	)
 	(gr_line
-		(start 78.41 101.03)
+		(start 78.41 97.982)
 		(end 78.41 106.11)
 		(stroke
@@
 		(layer "Edge.Cuts")
 	)
-	(gr_arc
-		(start 77.775 90.1334)
-		(mid 78.332962 88.786362)
-		(end 79.68 88.2284)
+	(gr_line
+		(start 77.774916 96.958675)
+		(end 77.775 90.1334)
 		(stroke
 			(width 0.15)
@@
 		(layer "Edge.Cuts")
 	)
-	(gr_line
-		(start 77.775 99.6584)
-		(end 77.775 90.1334)
+	(gr_arc
+		(start 77.775 90.1334)
+		(mid 78.332962 88.786362)
+		(end 79.68 88.2284)
 		(stroke
 			(width 0.15)
@@
 	)
 	(gr_arc
-		(start 79.045 99.6584)
-		(mid 78.41 100.2934)
-		(end 77.775 99.6584)
+		(start 79.045 96.951341)
+		(mid 78.41 97.586341)
+		(end 77.775 96.951341)
 		(stroke
 			(width 0.15)
@@
 	)
 	(gr_line
-		(start 79.045 99.6584)
+		(start 79.045 96.951341)
 		(end 79.045 90.1334)
 		(stroke
@@
 	)
 	(segment
+		(start 197.404 58.739)
+		(end 193.726 58.739)
+		(width 0.508)
+		(layer "F.Cu")
+		(net "/CTL_H")
+	)
+	(segment
 		(start 197.47 58.805)
 		(end 197.404 58.739)
@@
 	)
 	(segment
+		(start 193.789 58.802)
+		(end 193.726 58.739)
+		(width 0.508)
+		(layer "F.Cu")
+		(net "/CTL_H")
+	)
+	(segment
 		(start 144.958 53.786)
 		(end 141.656 53.786)
@@
 	)
 	(segment
-		(start 197.404 58.739)
+		(start 193.726 58.739)
 		(end 182.931 58.739)
 		(width 0.508)
@@
 	)
 	(segment
-		(start 193.789 58.802)
-		(end 193.789 61.152)
+		(start 193.789 61.152)
+		(end 193.789 58.802)
 		(width 0.508)
 		(layer "F.Cu")
@@
 	)
 	(segment
-		(start 193.726 58.739)
-		(end 193.789 58.802)
-		(width 0.508)
-		(layer "F.Cu")
-		(net "/CTL_H")
-	)
-	(segment
 		(start 141.656 53.786)
 		(end 141.275 54.167)
@@
 	)
 	(segment
-		(start 47.295 65.465)
-		(end 69.769 65.465)
-		(width 0.2032)
-		(layer "F.Cu")
-		(net "/CLK")
-	)
-	(segment
 		(start 167.3416 54.8336)
 		(end 168.453 55.945)
@@
 		(members "2556d83f-39ad-44f6-a1fc-b0d1fad3f834" "33f982ae-4567-40eb-90f8-2d074370fbb8"
 			"52621975-5b77-4261-b213-26dabe2c0b71" "532d3134-e727-4dea-bc9f-579412c9c937"
-			"73787d3c-3caa-4a5c-83ae-8473e2b8aaf1" "e25f31ad-84fb-4beb-9982-767f294b1c16"
-			"eb003e53-da21-4fc9-8f9c-ed8b2731cb21" "f61e856c-6b65-4783-92e3-2a0b5e25f517"
+			"73787d3c-3caa-4a5c-83ae-8473e2b8aaf1" "c5fe8924-e0a3-434d-a579-7d1afd7a2f85"
+			"e25f31ad-84fb-4beb-9982-767f294b1c16" "f61e856c-6b65-4783-92e3-2a0b5e25f517"
 		)
 	)

Commit message: [fp][rs] Change hole footprints to no soldermask
Parts:
- H1, H2, H3, H4, H5: footprint MountingHole:MountingHole_3.2mm_M3 -> CUSTOM:MountingHole_3.2mm_M3

Commit message: [rs] Check/Finalize PCB; Export gerbers v1.0A0
Parts:
- H3, H5: footprint CUSTOM:MountingHole_3.2mm_M3 -> MountingHole:MountingHole_3.2mm_M3_ISO14580_Pad_TopBottom
- H4: footprint CUSTOM:MountingHole_3.2mm_M3 -> MountingHole:MountingHole_3.2mm_M3_DIN965_Pad_TopBottom
- moved LAY1 1.78 mm to (44.8, 100.1)
Routing:
- net /CLK: track 133.5 -> 155.9 mm
- net /NEUTRAL: track 26.2 -> 28.6 mm
Other:
- board text added: "LD"
- board text added: "PWR"
